Commit message: Adjusted ex03

File: module_5/ex03/robot.gazebo.xacro (robot description, xacro)
@@ -4,18 +4,26 @@
   <gazebo reference="base_link">
     <material>Gazebo/Blue</material>
+    <mu1>0.2</mu1>
+    <mu2>0.2</mu2>
   </gazebo>
   <gazebo reference="left_wheel">
     <material>Gazebo/Black</material>
+    <mu1>1.0</mu1>
+    <mu2>1.0</mu2>
   </gazebo>
   <gazebo reference="right_wheel">
     <material>Gazebo/Black</material>
+    <mu1>1.0</mu1>
+    <mu2>1.0</mu2>
   </gazebo>
   <gazebo reference="caster_wheel">
     <material>Gazebo/Grey</material>
+    <mu1>0.5</mu1>
+    <mu2>0.5</mu2>
   </gazebo>
   <gazebo reference="sensor_tower">
     <material>Gazebo/Grey</material>
   </gazebo>
-  <!-- Differential Drive Controller -->
+  <!-- Differential Drive Controller - ПРОСТАЯ КОНФИГУРАЦИЯ -->
   <gazebo>
     <plugin filename="libgz-sim-diff-drive-system.so" name="gz::sim::systems::DiffDrive">
@@ -24,5 +32,6 @@
       <wheel_separation>1.2</wheel_separation>
       <wheel_radius>0.3</wheel_radius>
-      <odom_publish_frequency>30</odom_publish_frequency>
+      <max_linear_velocity>2.0</max_linear_velocity>
+      <max_angular_velocity>4.0</max_angular_velocity>
       <topic>cmd_vel</topic>
     </plugin>

File: module_5/ex03/robot.urdf.xacro (robot description, xacro)
@@ -19,7 +19,4 @@
   <xacro:property name="tower_radius" value="0.1" />
   <xacro:property name="tower_mass" value="3.0" />
-  <!-- Joint Limits -->
-  <xacro:property name="wheel_lower_limit" value="-10.0" />
-  <xacro:property name="wheel_upper_limit" value="10.0" />
   <!-- Colors -->
   <xacro:property name="blue_color" value="0.0 0.0 0.8 1.0" />
@@ -36,129 +33,131 @@
     <color rgba="${gray_color}" />
   </material>
-  <!-- Macro for creating a cylinder link -->
-  <xacro:macro name="cylinder_link" params="name radius length mass color xyz:='0 0 0' rpy:='0 0 0'">
-    <link name="${name}">
-      <visual>
-        <geometry>
-          <cylinder length="${length}" radius="${radius}" />
-        </geometry>
-        <material name="${color}" />
-        <origin xyz="${xyz}" rpy="${rpy}" />
-      </visual>
-      <collision>
-        <geometry>
-          <cylinder length="${length}" radius="${radius}" />
-        </geometry>
-        <origin xyz="${xyz}" rpy="${rpy}" />
-      </collision>
-      <inertial>
-        <mass value="${mass}" />
-        <inertia ixx="${mass * (3*radius*radius + length*length) / 12}"
-                 ixy="0.0"
-                 ixz="0.0"
-                 iyy="${mass * (3*radius*radius + length*length) / 12}"
-                 iyz="0.0"
-                 izz="${mass * radius*radius / 2}" />
-      </inertial>
-    </link>
-  </xacro:macro>
-  <!-- Macro for creating a sphere link -->
-  <xacro:macro name="sphere_link" params="name radius mass color">
-    <link name="${name}">
-      <visual>
-        <geometry>
-          <sphere radius="${radius}" />
-        </geometry>
-        <material name="${color}" />
-      </visual>
-      <collision>
-        <geometry>
-          <sphere radius="${radius}" />
-        </geometry>
-      </collision>
-      <inertial>
-        <mass value="${mass}" />
-        <inertia ixx="${2 * mass * radius * radius / 5}"
-                 ixy="0.0"
-                 ixz="0.0"
-                 iyy="${2 * mass * radius * radius / 5}"
-                 iyz="0.0"
-                 izz="${2 * mass * radius * radius / 5}" />
-      </inertial>
-    </link>
-  </xacro:macro>
-  <!-- Macro for creating a wheel joint -->
-  <xacro:macro name="wheel_joint" params="name parent child xyz">
-    <joint name="${name}" type="continuous">
-      <parent link="${parent}" />
-      <child link="${child}" />
-      <origin xyz="${xyz}" rpy="0 0 0" />
-      <axis xyz="0 1 0" />
-      <limit effort="10.0" velocity="5.0" />
-      <dynamics damping="0.1" friction="0.5" />
-    </joint>
-  </xacro:macro>
-  <!-- Macro for creating a fixed joint -->
-  <xacro:macro name="fixed_joint" params="name parent child xyz">
-    <joint name="${name}" type="fixed">
-      <parent link="${parent}" />
-      <child link="${child}" />
-      <origin xyz="${xyz}" rpy="0 0 0" />
-    </joint>
-  </xacro:macro>
   <!-- Base Link -->
-  <xacro:cylinder_link name="base_link"
-                       radius="${base_radius}"
-                       length="${base_height}"
-                       mass="${base_mass}"
-                       color="blue"
-                       xyz="0 0 ${base_height/2}" />
+  <link name="base_link">
+    <visual>
+      <geometry>
+        <cylinder length="${base_height}" radius="${base_radius}"/>
+      </geometry>
+      <material name="blue"/>
+      <origin xyz="0 0 ${base_height/2}" rpy="0 0 0"/>
+    </visual>
+    <collision>
+      <geometry>
+        <cylinder length="${base_height}" radius="${base_radius}"/>
+      </geometry>
+      <origin xyz="0 0 ${base_height/2}" rpy="0 0 0"/>
+    </collision>
+    <inertial>
+      <mass value="${base_mass}"/>
+      <inertia ixx="2.5" ixy="0.0" ixz="0.0" iyy="2.5" iyz="0.0" izz="1.5"/>
+    </inertial>
+  </link>
   <!-- Left Wheel -->
-  <xacro:cylinder_link name="left_wheel"
-                       radius="${wheel_radius}"
-                       length="${wheel_length}"
-                       mass="${wheel_mass}"
-                       color="black"
-                       rpy="${M_PI/2} 0 0" />
+  <link name="left_wheel">
+    <visual>
+      <geometry>
+        <cylinder length="${wheel_length}" radius="${wheel_radius}"/>
+      </geometry>
+      <material name="black"/>
+      <origin xyz="0 0 0" rpy="${M_PI/2} 0 0"/>
+    </visual>
+    <collision>
+      <geometry>
+        <cylinder length="${wheel_length}" radius="${wheel_radius}"/>
+      </geometry>
+      <origin xyz="0 0 0" rpy="${M_PI/2} 0 0"/>
+    </collision>
+    <inertial>
+      <mass value="${wheel_mass}"/>
+      <inertia ixx="0.1" ixy="0.0" ixz="0.0" iyy="0.1" iyz="0.0" izz="0.2"/>
+    </inertial>
+  </link>
   <!-- Right Wheel -->
-  <xacro:cylinder_link name="right_wheel"
-                       radius="${wheel_radius}"
-                       length="${wheel_length}"
-                       mass="${wheel_mass}"
-                       color="black"
-                       rpy="${M_PI/2} 0 0" />
+  <link name="right_wheel">
+    <visual>
+      <geometry>
+        <cylinder length="${wheel_length}" radius="${wheel_radius}"/>
+      </geometry>
+      <material name="black"/>
+      <origin xyz="0 0 0" rpy="${M_PI/2} 0 0"/>
+    </visual>
+    <collision>
+      <geometry>
+        <cylinder length="${wheel_length}" radius="${wheel_radius}"/>
+      </geometry>
+      <origin xyz="0 0 0" rpy="${M_PI/2} 0 0"/>
+    </collision>
+    <inertial>
+      <mass value="${wheel_mass}"/>
+      <inertia ixx="0.1" ixy="0.0" ixz="0.0" iyy="0.1" iyz="0.0" izz="0.2"/>
+    </inertial>
+  </link>
   <!-- Caster Wheel -->
-  <xacro:sphere_link name="caster_wheel"
-                     radius="${caster_radius}"
-                     mass="${caster_mass}"
-                     color="gray" />
+  <link name="caster_wheel">
+    <visual>
+      <geometry>
+        <sphere radius="${caster_radius}"/>
+      </geometry>
+      <material name="gray"/>
+    </visual>
+    <collision>
+      <geometry>
+        <sphere radius="${caster_radius}"/>
+      </geometry>
+    </collision>
+    <inertial>
+      <mass value="${caster_mass}"/>
+      <inertia ixx="0.01" ixy="0.0" ixz="0.0" iyy="0.01" iyz="0.0" izz="0.01"/>
+    </inertial>
+  </link>
   <!-- Sensor Tower -->
-  <xacro:cylinder_link name="sensor_tower"
-                       radius="${tower_radius}"
-                       length="${tower_height}"
-                       mass="${tower_mass}"
-                       color="gray"
-                       xyz="0 0 ${tower_height/2}" />
+  <link name="sensor_tower">
+    <visual>
+      <geometry>
+        <cylinder length="${tower_height}" radius="${tower_radius}"/>
+      </geometry>
+      <material name="gray"/>
+      <origin xyz="0 0 ${tower_height/2}" rpy="0 0 0"/>
+    </visual>
+    <collision>
+      <geometry>
+        <cylinder length="${tower_height}" radius="${tower_radius}"/>
+      </geometry>
+      <origin xyz="0 0 ${tower_height/2}" rpy="0 0 0"/>
+    </collision>
+    <inertial>
+      <mass value="${tower_mass}"/>
+      <inertia ixx="0.05" ixy="0.0" ixz="0.0" iyy="0.05" iyz="0.0" izz="0.02"/>
+    </inertial>
+  </link>
   <!-- Joints -->
   <!-- Left Wheel Joint -->
-  <xacro:wheel_joint name="left_wheel_joint"
-                     parent="base_link"
-                     child="left_wheel"
-                     xyz="-0.1 ${wheel_y_offset} ${wheel_z_offset}" />
+  <joint name="left_wheel_joint" type="continuous">
+    <parent link="base_link"/>
+    <child link="left_wheel"/>
+    <origin xyz="-0.1 ${wheel_y_offset} ${wheel_z_offset}" rpy="0 0 0"/>
+    <axis xyz="0 1 0"/>
+    <dynamics damping="0.1" friction="0.5"/>
+  </joint>
   <!-- Right Wheel Joint -->
-  <xacro:wheel_joint name="right_wheel_joint"
-                     parent="base_link"
-                     child="right_wheel"
-                     xyz="-0.1 -${wheel_y_offset} ${wheel_z_offset}" />
+  <joint name="right_wheel_joint" type="continuous">
+    <parent link="base_link"/>
+    <child link="right_wheel"/>
+    <origin xyz="-0.1 -${wheel_y_offset} ${wheel_z_offset}" rpy="0 0 0"/>
+    <axis xyz="0 1 0"/>
+    <dynamics damping="0.1" friction="0.5"/>
+  </joint>
   <!-- Caster Wheel Joint -->
-  <xacro:fixed_joint name="caster_wheel_joint"
-                     parent="base_link"
-                     child="caster_wheel"
-                     xyz="${caster_x_offset} 0 ${caster_z_offset}" />
+  <joint name="caster_wheel_joint" type="fixed">
+    <parent link="base_link"/>
+    <child link="caster_wheel"/>
+    <origin xyz="${caster_x_offset} 0 ${caster_z_offset}" rpy="0 0 0"/>
+  </joint>
   <!-- Sensor Tower Joint -->
-  <xacro:fixed_joint name="sensor_tower_joint"
-                     parent="base_link"
-                     child="sensor_tower"
-                     xyz="0 0 ${base_height}" />
+  <joint name="sensor_tower_joint" type="fixed">
+    <parent link="base_link"/>
+    <child link="sensor_tower"/>
+    <origin xyz="0 0 ${base_height}" rpy="0 0 0"/>
+  </joint>
   <!-- Gazebo plugins and extensions -->
   <xacro:include filename="$(find diff_drive_gazebo)/urdf/robot.gazebo.xacro" />
